File: dual_fan_control.kicad_pcb (KiCad board)
At the start: 2 copper layers, 50 x 50 mm, 77 parts, among them J1 UPDI, J2 FAN_4P, J3 FAN_4P, J4 PWR_SELECT, J5 Barrel_Jack_Switch, J6 USB_C_Receptacle_USB2.0, Q1 2N7002, Q2 AO4805, Q3 2N7002, Q4 AO4805, Q5 2N7002, SW1 SW_Push, SW2 SW_Push, SW3 PD_SEL, U1 ET6226M, U2 ATtiny1616-M, U3 TPS54202DDC, U4 CH224K

Commit message: Minor adjustments
Parts:
- H1, H2, H3: value MountingHole -> MountingHole_Pad; footprint MountingHole:MountingHole_2mm -> MountingHole:MountingHole_2.2mm_M2_DIN965_Pad
- J5: footprint Connector_BarrelJack:BarrelJack_Horizontal -> dual_fan_control:BarrelJack_Horizontal_CircularHoles
- moved H1 43.9 mm to (118.7, 55.9)
- moved H3 43.1 mm to (161.7, 54.5)
- moved H2 0.30 mm to (132.0, 90.5)
- moved J6 0.16 mm to (120.1, 64.1)
Routing:
- net GND: track 44.7 -> 48.0 mm, vias 47 -> 46
- net VDD: track 124.9 -> 124.3 mm
Other:
- board text added: "!"
- board text added: "0 1 0 0 1"
- board text added: "0 1 1 0 0"
- board text added: "0 1 1 1 1"
- board text added: "1"
- board text added: "2"
- board text added: "3"
- board text added: "5V 9V 12V 15V 20V"
- board text added: "PD"
- board text added: "SW3"
- board text added: "Set Correct PD Voltage First!"
- board text added: "UP = 1 DN = 0"
- board text added: "[4A]"
