File: dual_fan_control.kicad_pcb (KiCad board)
At the start: 2 copper layers, 50 x 50 mm, 77 parts, among them J1 UPDI, J2 FAN_4P, J3 FAN_4P, J4 PWR_SELECT, J5 Barrel_Jack_Switch, J6 USB_C_Receptacle_USB2.0, Q1 2N7002, Q2 AO4805, Q3 2N7002, Q4 AO4805, Q5 2N7002, SW1 SW_Push, SW2 SW_Push, SW3 PD_SEL, U1 ET6226M, U2 ATtiny1616-M, U3 TPS54202DDC, U4 CH224K

Commit message: Update IBOM
Parts:
- added G***: LOGO, slp_logo:sleepylogo_10mm, F.Cu at (122.2, 76.4)
- C6, C8, C9: footprint Capacitor_SMD:C_1206_3216Metric -> Capacitor_SMD:C_1210_3225Metric
- G***: moved to B.Cu
- moved C8 1.02 mm to (156.5, 54.7)
- moved L1 0.50 mm to (160.8, 48.7)
- moved C9 0.36 mm to (153.1, 54.7)
- moved C6 0.30 mm to (155.8, 48.2)
- turned G*** to 180 degrees
Routing:
- net GND: track 48.0 -> 49.4 mm
- net Net-(C5-Pad2): track 14.3 -> 14.8 mm

Commit message: Fix incorrect button net labels
Connections:
- R3 pad 2: BTN_ON -> BTN_SEL
- R6 pad 2: BTN_SEL -> BTN_ON
- SW1 pad 2: BTN_ON -> BTN_SEL
- SW2 pad 2: BTN_SEL -> BTN_ON
- U2 pad 13: BTN_ON -> BTN_SEL
- U2 pad 14: BTN_SEL -> BTN_ON
Routing:
- net BTN_SEL: track 17.0 -> 12.7 mm
- net BTN_ON: track 12.7 -> 17.0 mm
Changed lines of the file:
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@@
       (net 2 "GND") (pinfunction "1") (pintype "passive"))
     (pad "2" smd rect (at 3.9 0 180) (size 1.5 1.5) (layers "F.Cu" "F.Paste" "F.Mask")
-      (net 35 "BTN_ON") (pinfunction "2") (pintype "passive"))
+      (net 40 "BTN_SEL") (pinfunction "2") (pintype "passive"))
     (model "${KICAD6_3DMODEL_DIR}/Button_Switch_SMD.3dshapes/SW_SPST_CK_RS282G05A3.wrl"
       (offset (xyz 0 0 0))
@@
       (net 2 "GND") (pinfunction "1") (pintype "passive"))
     (pad "2" smd rect (at 3.9 0 180) (size 1.5 1.5) (layers "F.Cu" "F.Paste" "F.Mask")
-      (net 40 "BTN_SEL") (pinfunction "2") (pintype "passive"))
+      (net 35 "BTN_ON") (pinfunction "2") (pintype "passive"))
     (model "${KICAD6_3DMODEL_DIR}/Button_Switch_SMD.3dshapes/SW_SPST_CK_RS282G05A3.wrl"
       (offset (xyz 0 0 0))
@@
       (net 41 "LED_BOTH") (pinfunction "PB2") (pintype "bidirectional"))
     (pad "13" smd roundrect (at 1.45 0) (size 0.8 0.2) (layers "B.Cu" "B.Paste" "B.Mask") (roundrect_rratio 0.25)
-      (net 35 "BTN_ON") (pinfunction "PB1") (pintype "bidirectional"))
+      (net 40 "BTN_SEL") (pinfunction "PB1") (pintype "bidirectional"))
     (pad "14" smd roundrect (at 1.45 0.4) (size 0.8 0.2) (layers "B.Cu" "B.Paste" "B.Mask") (roundrect_rratio 0.25)
-      (net 40 "BTN_SEL") (pinfunction "PB0") (pintype "bidirectional"))
+      (net 35 "BTN_ON") (pinfunction "PB0") (pintype "bidirectional"))
     (pad "15" smd custom (at 1.45 0.8) (size 0.143431 0.143431) (layers "B.Cu" "B.Paste" "B.Mask")
       (net 39 "LED_FAN2") (pinfunction "PC0") (pintype "bidirectional")
@@
       (net 1 "VDD") (pintype "passive"))
     (pad "2" smd roundrect (at 0.825 0 270) (size 0.8 0.95) (layers "B.Cu" "B.Paste" "B.Mask") (roundrect_rratio 0.25)
-      (net 40 "BTN_SEL") (pintype "passive"))
+      (net 35 "BTN_ON") (pintype "passive"))
     (model "${KICAD6_3DMODEL_DIR}/Resistor_SMD.3dshapes/R_0603_1608Metric.wrl"
       (offset (xyz 0 0 0))
@@
       (net 1 "VDD") (pintype "passive"))
     (pad "2" smd roundrect (at 0.825 0 270) (size 0.8 0.95) (layers "B.Cu" "B.Paste" "B.Mask") (roundrect_rratio 0.25)
-      (net 35 "BTN_ON") (pintype "passive"))
+      (net 40 "BTN_SEL") (pintype "passive"))
     (model "${KICAD6_3DMODEL_DIR}/Resistor_SMD.3dshapes/R_0603_1608Metric.wrl"
       (offset (xyz 0 0 0))
@@
   (segment (start 150.6 85.8) (end 152.6 85.8) (width 0.2) (layer "B.Cu") (net 34))
   (segment (start 152.6 85.8) (end 152.85 85.55) (width 0.2) (layer "B.Cu") (net 34))
-  (segment (start 154.95 86.15) (end 154 85.2) (width 0.25) (layer "F.Cu") (net 35))
-  (segment (start 157.1 86.15) (end 154.95 86.15) (width 0.25) (layer "F.Cu") (net 35))
-  (segment (start 154 85.2) (end 154 84.2) (width 0.25) (layer "F.Cu") (net 35))
-  (via (at 157.1 86.15) (size 0.8) (drill 0.4) (layers "F.Cu" "B.Cu") (net 35))
-  (segment (start 155.45 89) (end 151.95 89) (width 0.2) (layer "B.Cu") (net 35))
-  (segment (start 157.1 86.15) (end 157.1 87.35) (width 0.2) (layer "B.Cu") (net 35))
-  (segment (start 157.1 86.15) (end 157.1 85.025) (width 0.25) (layer "B.Cu") (net 35))
-  (segment (start 157.1 87.35) (end 155.45 89) (width 0.2) (layer "B.Cu") (net 35))
+  (segment (start 158.4 89.6) (end 154 89.6) (width 0.25) (layer "F.Cu") (net 35))
+  (segment (start 158.8 89.2) (end 158.4 89.6) (width 0.25) (layer "F.Cu") (net 35))
+  (segment (start 158.8 86.9) (end 158.8 89.2) (width 0.25) (layer "F.Cu") (net 35))
+  (via (at 158.8 86.9) (size 0.8) (drill 0.4) (layers "F.Cu" "B.Cu") (net 35))
+  (segment (start 156.3 89.4) (end 158.8 86.9) (width 0.2) (layer "B.Cu") (net 35))
+  (segment (start 151.95 89.4) (end 156.3 89.4) (width 0.2) (layer "B.Cu") (net 35))
+  (segment (start 158.8 86.9) (end 158.8 85.025) (width 0.25) (layer "B.Cu") (net 35))
   (segment (start 150.8 86.3) (end 153.2 86.3) (width 0.2) (layer "B.Cu") (net 36))
   (segment (start 153.7 85.8) (end 153.7 85.025) (width 0.2) (layer "B.Cu") (net 36))
@@
   (segment (start 157.3 89.8) (end 160.5 86.6) (width 0.2) (layer "B.Cu") (net 39))
   (segment (start 160.5 86.6) (end 160.5 85.025) (width 0.2) (layer "B.Cu") (net 39))
-  (segment (start 158.4 89.6) (end 154 89.6) (width 0.25) (layer "F.Cu") (net 40))
-  (segment (start 158.8 89.2) (end 158.4 89.6) (width 0.25) (layer "F.Cu") (net 40))
-  (segment (start 158.8 86.9) (end 158.8 89.2) (width 0.25) (layer "F.Cu") (net 40))
-  (via (at 158.8 86.9) (size 0.8) (drill 0.4) (layers "F.Cu" "B.Cu") (net 40))
-  (segment (start 156.3 89.4) (end 158.8 86.9) (width 0.2) (layer "B.Cu") (net 40))
-  (segment (start 151.95 89.4) (end 156.3 89.4) (width 0.2) (layer "B.Cu") (net 40))
-  (segment (start 158.8 86.9) (end 158.8 85.025) (width 0.25) (layer "B.Cu") (net 40))
+  (segment (start 154.95 86.15) (end 154 85.2) (width 0.25) (layer "F.Cu") (net 40))
+  (segment (start 157.1 86.15) (end 154.95 86.15) (width 0.25) (layer "F.Cu") (net 40))
+  (segment (start 154 85.2) (end 154 84.2) (width 0.25) (layer "F.Cu") (net 40))
+  (via (at 157.1 86.15) (size 0.8) (drill 0.4) (layers "F.Cu" "B.Cu") (net 40))
+  (segment (start 155.45 89) (end 151.95 89) (width 0.2) (layer "B.Cu") (net 40))
+  (segment (start 157.1 86.15) (end 157.1 87.35) (width 0.2) (layer "B.Cu") (net 40))
+  (segment (start 157.1 86.15) (end 157.1 85.025) (width 0.25) (layer "B.Cu") (net 40))
+  (segment (start 157.1 87.35) (end 155.45 89) (width 0.2) (layer "B.Cu") (net 40))
   (segment (start 151.95 88.6) (end 154.7 88.6) (width 0.2) (layer "B.Cu") (net 41))
   (segment (start 154.7 88.6) (end 155.4 87.9) (width 0.2) (layer "B.Cu") (net 41))
