File: dual_fan_control.kicad_sch (KiCad schematic)
At the start: 76 parts, among them J1 UPDI, J2 FAN_4P, J3 FAN_4P, J4 PWR_SELECT, J5 Barrel_Jack_Switch, J6 USB_C_Receptacle_USB2.0, Q1 2N7002, Q2 AO4805, Q3 2N7002, Q4 AO4805, Q5 2N7002, SW1 SW_Push, SW2 SW_Push, SW3 PD_SEL, U1 ET6226M, U2 ATtiny1616-M, U3 TPS54202DDC, U4 CH224K

Commit message: Minor adjustments
Parts:
- removed H1, H2, H3: MountingHole, MountingHole:MountingHole_2mm, symbol Mechanical:MountingHole
- added H1, H2, H3: MountingHole_Pad, MountingHole:MountingHole_2.2mm_M2_DIN965_Pad, symbol Mechanical:MountingHole_Pad
- J5: footprint Connector_BarrelJack:BarrelJack_Horizontal -> dual_fan_control:BarrelJack_Horizontal_CircularHoles
Connections:
- no-connect marks 11 -> 14
Changed lines of the file:
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@@
   (no_connect (at 39.37 59.69))
   (no_connect (at 55.88 238.76))
+  (no_connect (at 45.72 101.6))
+  (no_connect (at 68.58 101.6))
+  (no_connect (at 91.44 101.6))
   (no_connect (at 55.88 236.22))
   (no_connect (at 43.18 173.99))
@@
     (pin "2")
   )
-  (symbol (lib_id "Mechanical:MountingHole") (at 60.96 97.79 0) (unit 1)
-    (in_bom yes) (on_board yes) (fields_autoplaced)
-    (property "Reference" "H2" (id 0) (at 63.5 96.5199 0)
-      (effects (font (size 1.27 1.27)) (justify left))
-    )
-    (property "Value" "MountingHole" (id 1) (at 63.5 99.0599 0)
-      (effects (font (size 1.27 1.27)) (justify left))
-    )
-    (property "Footprint" "MountingHole:MountingHole_2mm" (id 2) (at 60.96 97.79 0)
-      (effects (font (size 1.27 1.27)) hide)
-    )
-    (property "Datasheet" "~" (id 3) (at 60.96 97.79 0)
-      (effects (font (size 1.27 1.27)) hide)
-    )
-  )
   (symbol (lib_id "Transistor_FET:2N7002") (at 167.64 231.14 0) (unit 1)
     (in_bom yes) (on_board yes) (fields_autoplaced)
@@
     (pin "1")
   )
-  (symbol (lib_id "Mechanical:MountingHole") (at 41.91 97.79 0) (unit 1)
-    (in_bom yes) (on_board yes) (fields_autoplaced)
-    (property "Reference" "H1" (id 0) (at 44.45 96.5199 0)
-      (effects (font (size 1.27 1.27)) (justify left))
-    )
-    (property "Value" "MountingHole" (id 1) (at 44.45 99.0599 0)
-      (effects (font (size 1.27 1.27)) (justify left))
-    )
-    (property "Footprint" "MountingHole:MountingHole_2mm" (id 2) (at 41.91 97.79 0)
-      (effects (font (size 1.27 1.27)) hide)
-    )
-    (property "Datasheet" "~" (id 3) (at 41.91 97.79 0)
-      (effects (font (size 1.27 1.27)) hide)
-    )
-  )
   (symbol (lib_id "power:VDD") (at 153.67 35.56 0) (unit 1)
     (in_bom yes) (on_board yes) (fields_autoplaced)
@@
     (property "Reference" "J5" (id 0) (at 35.56 165.1 0))
     (property "Value" "Barrel_Jack_Switch" (id 1) (at 35.56 167.64 0))
-    (property "Footprint" "Connector_BarrelJack:BarrelJack_Horizontal" (id 2) (at 36.83 175.006 0)
+    (property "Footprint" "dual_fan_control:BarrelJack_Horizontal_CircularHoles" (id 2) (at 36.83 175.006 0)
       (effects (font (size 1.27 1.27)) hide)
     )
@@
     (pin "2")
   )
+  (symbol (lib_id "Mechanical:MountingHole_Pad") (at 45.72 99.06 0) (unit 1)
+    (in_bom yes) (on_board yes) (fields_autoplaced)
+    (property "Reference" "H1" (id 0) (at 48.26 96.5199 0)
+      (effects (font (size 1.27 1.27)) (justify left))
+    )
+    (property "Value" "MountingHole_Pad" (id 1) (at 48.26 99.0599 0)
+      (effects (font (size 1.27 1.27)) (justify left))
+    )
+    (property "Footprint" "MountingHole:MountingHole_2.2mm_M2_DIN965_Pad" (id 2) (at 45.72 99.06 0)
+      (effects (font (size 1.27 1.27)) hide)
+    )
+    (property "Datasheet" "~" (id 3) (at 45.72 99.06 0)
+      (effects (font (size 1.27 1.27)) hide)
+    )
+    (pin "1")
+  )
   (symbol (lib_id "Device:C_Small") (at 83.82 119.38 90) (unit 1)
     (in_bom yes) (on_board yes) (fields_autoplaced)
@@
     (pin "2")
   )
+  (symbol (lib_id "Mechanical:MountingHole_Pad") (at 91.44 99.06 0) (unit 1)
+    (in_bom yes) (on_board yes) (fields_autoplaced)
+    (property "Reference" "H3" (id 0) (at 93.98 96.5199 0)
+      (effects (font (size 1.27 1.27)) (justify left))
+    )
+    (property "Value" "MountingHole_Pad" (id 1) (at 93.98 99.0599 0)
+      (effects (font (size 1.27 1.27)) (justify left))
+    )
+    (property "Footprint" "MountingHole:MountingHole_2.2mm_M2_DIN965_Pad" (id 2) (at 91.44 99.06 0)
+      (effects (font (size 1.27 1.27)) hide)
+    )
+    (property "Datasheet" "~" (id 3) (at 91.44 99.06 0)
+      (effects (font (size 1.27 1.27)) hide)
+    )
+    (pin "1")
+  )
   (symbol (lib_id "Device:R_Small") (at 137.16 38.1 90) (unit 1)
     (in_bom yes) (on_board yes) (fields_autoplaced)
@@
     (pin "2")
   )
+  (symbol (lib_id "Mechanical:MountingHole_Pad") (at 68.58 99.06 0) (unit 1)
+    (in_bom yes) (on_board yes) (fields_autoplaced)
+    (property "Reference" "H2" (id 0) (at 71.12 96.5199 0)
+      (effects (font (size 1.27 1.27)) (justify left))
+    )
+    (property "Value" "MountingHole_Pad" (id 1) (at 71.12 99.0599 0)
+      (effects (font (size 1.27 1.27)) (justify left))
+    )
+    (property "Footprint" "MountingHole:MountingHole_2.2mm_M2_DIN965_Pad" (id 2) (at 68.58 99.06 0)
+      (effects (font (size 1.27 1.27)) hide)
+    )
+    (property "Datasheet" "~" (id 3) (at 68.58 99.06 0)
+      (effects (font (size 1.27 1.27)) hide)
+    )
+    (pin "1")
+  )
   (symbol (lib_id "power:VDD") (at 278.13 49.53 0) (unit 1)
     (in_bom yes) (on_board yes) (fields_autoplaced)
@@
     (pin "2")
   )
-  (symbol (lib_id "Mechanical:MountingHole") (at 80.01 97.79 0) (unit 1)
-    (in_bom yes) (on_board yes) (fields_autoplaced)
-    (property "Reference" "H3" (id 0) (at 82.55 96.5199 0)
-      (effects (font (size 1.27 1.27)) (justify left))
-    )
-    (property "Value" "MountingHole" (id 1) (at 82.55 99.0599 0)
-      (effects (font (size 1.27 1.27)) (justify left))
-    )
-    (property "Footprint" "MountingHole:MountingHole_2mm" (id 2) (at 80.01 97.79 0)
-      (effects (font (size 1.27 1.27)) hide)
-    )
-    (property "Datasheet" "~" (id 3) (at 80.01 97.79 0)
-      (effects (font (size 1.27 1.27)) hide)
-    )
-  )
   (sheet_instances
     (path "/" (page "1"))
@@
       (reference "F1") (unit 1) (value "JK-MSMD200-24V") (footprint "Fuse:Fuse_1812_4532Metric_Pad1.30x3.40mm_HandSolder")
     )
-    (path "/62c89ae9-ec5e-472c-8fef-750bbb132580"
-      (reference "H1") (unit 1) (value "MountingHole") (footprint "MountingHole:MountingHole_2mm")
+    (path "/db3e3de3-5687-40b8-9114-d42e15c952ae"
+      (reference "H1") (unit 1) (value "MountingHole_Pad") (footprint "MountingHole:MountingHole_2.2mm_M2_DIN965_Pad")
     )
-    (path "/1cb9a905-150a-4971-bd8f-c63baad66e16"
-      (reference "H2") (unit 1) (value "MountingHole") (footprint "MountingHole:MountingHole_2mm")
+    (path "/ee616598-f860-4670-ae3e-8a8e50f73eb0"
+      (reference "H2") (unit 1) (value "MountingHole_Pad") (footprint "MountingHole:MountingHole_2.2mm_M2_DIN965_Pad")
     )
-    (path "/f84567e8-7501-4d55-8910-85ef6899eaa2"
-      (reference "H3") (unit 1) (value "MountingHole") (footprint "MountingHole:MountingHole_2mm")
+    (path "/dde07420-43eb-4327-87fc-bab504a9e95b"
+      (reference "H3") (unit 1) (value "MountingHole_Pad") (footprint "MountingHole:MountingHole_2.2mm_M2_DIN965_Pad")
     )
     (path "/682c52f5-a6c1-4d28-a680-46495fb98c8c"
@@
     )
     (path "/a7240828-6fc1-428b-8ef0-b57ce84d88a2"
-      (reference "J5") (unit 1) (value "Barrel_Jack_Switch") (footprint "Connector_BarrelJack:BarrelJack_Horizontal")
+      (reference "J5") (unit 1) (value "Barrel_Jack_Switch") (footprint "dual_fan_control:BarrelJack_Horizontal_CircularHoles")
     )
     (path "/781c55de-b229-47b4-9e37-8df961ca29ac"

Commit message: Update IBOM
Parts:
- C6, C8, C9: footprint Capacitor_SMD:C_1206_3216Metric -> Capacitor_SMD:C_1210_3225Metric
Changed lines of the file:
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@@
       (effects (font (size 1.27 1.27)) (justify left))
     )
-    (property "Footprint" "Capacitor_SMD:C_1206_3216Metric" (id 2) (at 101.6 125.73 0)
+    (property "Footprint" "Capacitor_SMD:C_1210_3225Metric" (id 2) (at 101.6 125.73 0)
       (effects (font (size 1.27 1.27)) hide)
     )
@@
       (effects (font (size 1.27 1.27)) (justify left))
     )
-    (property "Footprint" "Capacitor_SMD:C_1206_3216Metric" (id 2) (at 111.76 125.73 0)
+    (property "Footprint" "Capacitor_SMD:C_1210_3225Metric" (id 2) (at 111.76 125.73 0)
       (effects (font (size 1.27 1.27)) hide)
     )
@@
       (effects (font (size 1.27 1.27)) (justify left))
     )
-    (property "Footprint" "Capacitor_SMD:C_1206_3216Metric" (id 2) (at 36.83 123.19 0)
+    (property "Footprint" "Capacitor_SMD:C_1210_3225Metric" (id 2) (at 36.83 123.19 0)
       (effects (font (size 1.27 1.27)) hide)
     )
@@
     )
     (path "/805d2b98-a373-4477-9219-ae952529caf4"
-      (reference "C6") (unit 1) (value "22uF") (footprint "Capacitor_SMD:C_1206_3216Metric")
+      (reference "C6") (unit 1) (value "22uF") (footprint "Capacitor_SMD:C_1210_3225Metric")
     )
     (path "/367b0f0e-1b9f-4e0e-affa-12feaffd716b"
@@
     )
     (path "/417047ea-0e59-4614-a104-d6053a966837"
-      (reference "C8") (unit 1) (value "22uF") (footprint "Capacitor_SMD:C_1206_3216Metric")
+      (reference "C8") (unit 1) (value "22uF") (footprint "Capacitor_SMD:C_1210_3225Metric")
     )
     (path "/50c29b17-24c2-41a7-8b2a-a5d5690fd187"
-      (reference "C9") (unit 1) (value "22uF") (footprint "Capacitor_SMD:C_1206_3216Metric")
+      (reference "C9") (unit 1) (value "22uF") (footprint "Capacitor_SMD:C_1210_3225Metric")
     )
     (path "/890e7c73-f434-453f-9d32-1cbca387b59a"

Commit message: Fix incorrect button net labels
Connections:
- net BTN_ON: now also R6.2, SW2.2, U2.14 (PB0); no longer R3.2, SW1.2, U2.13 (PB1)
- net BTN_SEL: now also R3.2, SW1.2, U2.13 (PB1); no longer R6.2, SW2.2, U2.14 (PB0)
Changed lines of the file:
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@@
     )
   )
-  (global_label "BTN_ON" (shape output) (at 191.77 38.1 0) (fields_autoplaced)
+  (global_label "BTN_SEL" (shape output) (at 191.77 38.1 0) (fields_autoplaced)
     (effects (font (size 1.27 1.27)) (justify left))
-    (property "Intersheet References" "${INTERSHEET_REFS}" (id 0) (at 201.3798 38.0206 0)
+    (property "Intersheet References" "${INTERSHEET_REFS}" (id 0) (at 202.1055 38.0206 0)
       (effects (font (size 1.27 1.27)) (justify left) hide)
     )
@@
     )
   )
-  (global_label "BTN_SEL" (shape input) (at 72.39 54.61 0) (fields_autoplaced)
+  (global_label "BTN_ON" (shape input) (at 72.39 54.61 0) (fields_autoplaced)
     (effects (font (size 1.27 1.27)) (justify left))
-    (property "Intersheet References" "${INTERSHEET_REFS}" (id 0) (at 82.7255 54.5306 0)
+    (property "Intersheet References" "${INTERSHEET_REFS}" (id 0) (at 81.9998 54.5306 0)
       (effects (font (size 1.27 1.27)) (justify left) hide)
     )
@@
     )
   )
-  (global_label "BTN_SEL" (shape output) (at 191.77 64.77 0) (fields_autoplaced)
+  (global_label "BTN_ON" (shape output) (at 191.77 64.77 0) (fields_autoplaced)
     (effects (font (size 1.27 1.27)) (justify left))
-    (property "Intersheet References" "${INTERSHEET_REFS}" (id 0) (at 202.1055 64.6906 0)
+    (property "Intersheet References" "${INTERSHEET_REFS}" (id 0) (at 201.3798 64.6906 0)
       (effects (font (size 1.27 1.27)) (justify left) hide)
     )
   )
-  (global_label "BTN_ON" (shape input) (at 72.39 57.15 0) (fields_autoplaced)
+  (global_label "BTN_SEL" (shape input) (at 72.39 57.15 0) (fields_autoplaced)
     (effects (font (size 1.27 1.27)) (justify left))
-    (property "Intersheet References" "${INTERSHEET_REFS}" (id 0) (at 81.9998 57.0706 0)
+    (property "Intersheet References" "${INTERSHEET_REFS}" (id 0) (at 82.7255 57.0706 0)
       (effects (font (size 1.27 1.27)) (justify left) hide)
     )
